Commit message: sim: add camera + LIDAR sensors
Add forward-facing camera (640x480, 30Hz, ~1.2rad HFOV, ~20deg down
tilt) on the front bumper and 360-deg single-plane LIDAR (360 samples,
10m range, 10Hz) on top of the chassis. Camera publishes to /camera/*
via libgazebo_ros_camera; LIDAR publishes /scan via
libgazebo_ros_ray_sensor. camera_link_optical is added with the
standard optical-frame rotation so downstream perception can use it
directly for projection math.

Note on /camera namespace: <namespace>/</namespace> is set explicitly
inside the camera plugin <ros> block; without it, gazebo_ros_camera
stacks namespace+camera_name and topics end up at /camera/camera/*.

Verified: /scan steady 10.0Hz, /camera/image_raw ~8Hz with high
variance (rqt subscriber overhead, not sim — Gazebo RTF is 1.0).
Ticks Day 1 of PROGRESS.md.

File: urdf/mobile_arm.urdf.xacro (robot description, xacro)
@@ -239,4 +239,96 @@
   <xacro:finger prefix="right" sign="1"/>
   <!-- ============================================================== -->
+  <!-- Camera: forward-facing, 20° down tilt, on top of front bumper  -->
+  <!-- ============================================================== -->
+  <link name="camera_link">
+    <visual>
+      <origin xyz="0 0 0" rpy="0 0 0"/>
+      <geometry><box size="0.04 0.06 0.04"/></geometry>
+      <material name="black"/>
+    </visual>
+    <collision>
+      <origin xyz="0 0 0" rpy="0 0 0"/>
+      <geometry><box size="0.04 0.06 0.04"/></geometry>
+    </collision>
+    <xacro:box_inertia m="0.05" x="0.04" y="0.06" z="0.04"/>
+  </link>
+  <joint name="camera_joint" type="fixed">
+    <parent link="base_link"/>
+    <child  link="camera_link"/>
+    <origin xyz="0.20 0 0.18" rpy="0 0.349 0"/>
+  </joint>
+  <link name="camera_link_optical"/>
+  <joint name="camera_optical_joint" type="fixed">
+    <parent link="camera_link"/>
+    <child  link="camera_link_optical"/>
+    <origin xyz="0 0 0" rpy="${-pi/2} 0 ${-pi/2}"/>
+  </joint>
+  <gazebo reference="camera_link">
+    <material>Gazebo/FlatBlack</material>
+    <sensor type="camera" name="camera_sensor">
+      <update_rate>30.0</update_rate>
+      <camera>
+        <horizontal_fov>1.2</horizontal_fov>
+        <image><width>640</width><height>480</height><format>R8G8B8</format></image>
+        <clip><near>0.02</near><far>10</far></clip>
+      </camera>
+      <plugin name="camera_plugin" filename="libgazebo_ros_camera.so">
+        <ros><namespace>/</namespace></ros>
+        <camera_name>camera</camera_name>
+        <frame_name>camera_link_optical</frame_name>
+      </plugin>
+    </sensor>
+  </gazebo>
+  <!-- ============================================================== -->
+  <!-- LIDAR: 360° single-plane on top of chassis                     -->
+  <!-- ============================================================== -->
+  <link name="lidar_link">
+    <visual>
+      <origin xyz="0 0 0.02" rpy="0 0 0"/>
+      <geometry><cylinder length="0.04" radius="0.04"/></geometry>
+      <material name="black"/>
+    </visual>
+    <collision>
+      <origin xyz="0 0 0.02" rpy="0 0 0"/>
+      <geometry><cylinder length="0.04" radius="0.04"/></geometry>
+    </collision>
+    <xacro:cylinder_inertia m="0.1" r="0.04" h="0.04"/>
+  </link>
+  <joint name="lidar_joint" type="fixed">
+    <parent link="base_link"/>
+    <child  link="lidar_link"/>
+    <origin xyz="0 0 0.13" rpy="0 0 0"/>
+  </joint>
+  <gazebo reference="lidar_link">
+    <material>Gazebo/FlatBlack</material>
+    <sensor type="ray" name="lidar_sensor">
+      <pose>0 0 0.02 0 0 0</pose>
+      <update_rate>10</update_rate>
+      <ray>
+        <scan>
+          <horizontal>
+            <samples>360</samples>
+            <resolution>1</resolution>
+            <min_angle>-3.14159</min_angle>
+            <max_angle>3.14159</max_angle>
+          </horizontal>
+        </scan>
+        <range>
+          <min>0.10</min>
+          <max>10.0</max>
+          <resolution>0.01</resolution>
+        </range>
+      </ray>
+      <plugin name="lidar_plugin" filename="libgazebo_ros_ray_sensor.so">
+        <ros>
+          <namespace>/</namespace>
+          <remapping>~/out:=scan</remapping>
+        </ros>
+        <output_type>sensor_msgs/LaserScan</output_type>
+        <frame_name>lidar_link</frame_name>
+      </plugin>
+    </sensor>
+  </gazebo>
+  <!-- ============================================================== -->
   <!-- ros2_control: arm + gripper joints, position-commanded         -->
   <!-- ============================================================== -->
